File: scheme/game_pad_keyboard_v0.1/game_pad_keyboard.sch (KiCad schematic (older format))
At the start: 207 parts, among them J1 USB, J2 GPIO, J3 SWD, M1 vibrator, Q1 BSS138, Q2 BSS138, Q3 BSS138, Q4 BSS138, Q5 BSS138, Q6 BSS138, Q7 BSS138, Q8 BSS138, SW1 SW_Push, SW10 SW_Push, SW11 SW_Push, SW12 SW_Push, SW13 SW_Push, SW14 Reset, SW15 Battery, SW2 SW_Push, SW3 SW_Push, SW4 SW_Push, SW5 Power, SW6 SW_Push, SW7 SW_Push, SW8 SW_Push, SW9 SW_Push, U1 LM75B, U10 ADM3485, U11 NRF24L01_Breakout, U12 MAX3232, U13 CH340G, U14 JDY-23, U2 AMS1117-3.3, U3 DS3231M, U4 TP5400, U5 74HC595, U6 74HC595, U7 74HC595, U8 STM32F103C6Tx, U9 74HC165, Y1 8MHz, Y2 12MHz

Commit message: fix: Caps location
Location of the capacitors has changed; they are
now located after the transistors.
Parts:
- renumbered C18 to C17, C17 to C18
Connections:
- net +3V3: now also Q1.3 (D); no longer C17.1, C26.1, C27.1, C28.1, C34.1, C35.1, DS1.8 (LEDA)
- net GND: now also C26.1, C27.1, C28.1, C34.1, C35.1, DS1.9 (LEDK); no longer C26.2, C27.2, C28.2, C34.2, C35.2, Q1.2 (S)
- net at Q7.2 (S), U13.16 (VCC), U13.4 (V3): now also C34.2
- net at Q5.2 (S), U11.2 (VCC): now also C27.2
- net at Q4.2 (S), U10.8 (VCC): now also C26.2
- net at Q6.2 (S), U12.16 (VCC): now also C28.2
- net at Q8.2 (S), U14.1 (Vcc): now also C35.2
- removed net display_cathode: DS1.9 (LEDK), Q1.3 (D)
- new net display_anode: C17.1, DS1.8 (LEDA), Q1.2 (S)
Other:
- note removed: "r2r"
- moved on the sheet: BT1, C1, C12, C14, C16, C17, C18, C19, C21, C26, C27, C28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
